Commit message: rplidar mesh added

File: cpswarm_bringup/urdf/kobuki_gazebo.urdf.xacro (robot description, xacro)
@@ -162,7 +162,7 @@
 	  <gazebo>
 	    <plugin name="kobuki_controller" filename="libgazebo_ros_kobuki.so">
-		  <odom_frame>/${prefix_frame}odom</odom_frame>
-		  <base_link_frame>/${prefix_frame}base_link</base_link_frame>
-		  <base_footprint_frame>/${prefix_frame}base_footprint</base_footprint_frame>
+		  <odom_frame>${prefix_frame}odom</odom_frame>
+		  <base_link_frame>${prefix_frame}base_link</base_link_frame>
+		  <base_footprint_frame>${prefix_frame}base_footprint</base_footprint_frame>
 	      <publish_tf>1</publish_tf>
 	      <left_wheel_joint_name>${prefix_frame}wheel_left_joint</left_wheel_joint_name>
@@ -177,5 +177,6 @@
 	      <cliff_detection_threshold>0.04</cliff_detection_threshold>
 	      <bumper_name>bumpers</bumper_name>
-        <imu_name>/${prefix_frame}imu</imu_name>
+	      <ignoreTfPrefix>1</ignoreTfPrefix>
+        <imu_name>imu</imu_name>
 	    </plugin>
 	  </gazebo>

File: cpswarm_bringup/urdf/rplidar.urdf.xacro (robot description, xacro)
@@ -11,5 +11,5 @@
         <origin xyz="0 0 0" rpy="0 0 0"/>
         <geometry>
-            <mesh filename="package://turtlebot_description/meshes/sensors/rplidar.stl"/>
+            <mesh filename="package://cpswarm_bringup/meshes/sensors/rplidar.stl"/>
         </geometry>
       </collision>
@@ -17,5 +17,5 @@
         <origin xyz="0 0 0" rpy="${-M_PI/2} 0 0"/>
         <geometry>
-            <mesh filename="package://turtlebot_description/meshes/sensors/rplidar2.dae"/>
+            <mesh filename="package://cpswarm_bringup/meshes/sensors/rplidar.dae"/>
         </geometry>
       </visual>
