Commit message: xacro model updated

File: cpswarm_bringup/urdf/nostacks.urdf.xacro (robot description, xacro)
@@ -116,4 +116,9 @@
       <axis xyz="0 0 1"/>
     </joint>
+    <!--joint name="${prefix_frame}plate_middle_joint" type="fixed">
+      <origin xyz="-0.01364 0.0 0.1914" rpy="0 0 0"/>
+      <parent link="${parent}"/>
+      <child link="${prefix_frame}plate_middle_link"/>
+    </joint-->
     <link name="${prefix_frame}plate_middle_link">
       <visual>
@@ -152,5 +157,6 @@
     </collision>
   </gazebo>
-  <xacro:elevator_transmission prefix_frame="${prefix_frame}" />
+  <!--xacro:elevator_transmission prefix_frame="${prefix_frame}" /-->
+	<xacro:elevator_transmission prefix_frame="${prefix_frame}" />
   </xacro:macro>
 </robot>
